File: ra8p1_kicad/ereader/mcu_supply_power.kicad_sch (KiCad schematic)
At the start: 20 parts, among them U1 R7KA8P1KFLCAC#UC0

Commit message: feat(hardware): track schematic BOM and DigiKey sourcing risks
Parts:
- C16, C17, C18, C19, C20, C21, C22, C23, C24, C25, C26, C27, C28, C29, C30, C31, C32, C33, C34: Procurement_Status (none) -> TBD - exact MPN, ratings and DigiKey sourcing required
- U1: DigiKey_Part_Number (none) -> 559-R7KA8P1KFLCAC#UC0-ND; DigiKey_URL (none) -> https://www.digikey.com/en/products/detail/renesas-electron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; Procurement_Status (none) -> HOLD - DigiKey discontinued; qualify orderable RA8P1 suffix; Sourcing_Snapshot (none) -> 2026-09-05 indexed: stock 1; USD 29.47; no backorders. Dist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

Commit message: feat(hardware): add Mouser sourcing and qualify MCU pull-up resistors
Parts:
- U1: Mouser Part Number (none) -> 968-R7KA8P1KFLCACUC0; Mouser Price/Stock (none) -> 2026-09-05 browser: 317 in stock; USD 1:29.47 / 10:23.82 / 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; Mouser_URL (none) -> https://www.mouser.com/en/ProductDetail/Renesas-Electronics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; Procurement_Status HOLD - DigiKey discontinued; qualify orderable RA8P1 suffix -> Retain exact UC0 - Mouser stock verified; circuit qualifica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

Commit message: feat(hardware): source and screen MCU bypass capacitors
Parts:
- C16, C17, C18, C19, C20, C21, C22, C23, C24, C25, C26, C27, C28, C29, C30, C31, C32, C33, C34: DigiKey_Part_Number (none) -> 445-1314-1-ND; DigiKey_URL (none) -> https://www.digikey.com/en/products/detail/tdk-corporation/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; Manufacturer_Name (none) -> TDK; Manufacturer_Part_Number (none) -> C1608X7R1H104K080AA; Procurement_Status TBD - exact MPN, ratings and DigiKey sourcing required -> Selected - nominal DC-bias screened; final rail and PDN qua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; Selection_Basis (none) -> 100 nF +/-10%, 50 V X7R. +3V3_MCU bypass. TDK nominal DC-bi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; Sourcing_Snapshot (none) -> 2026-09-05: TDK Production; DigiKey Active, 374087 in stock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
