File: ra8p1_kicad/ereader/mcu_clocks_debug.kicad_sch (KiCad schematic)
At the start: 15 parts, among them J1 Cortex Debug 10-pin, SW1 RESET, SW2 BOOT, U1 R7KA8P1KFLCAC#UC0, Y1 24MHz, Y2 32.768kHz

Commit message: Add e-reader reset supervisor with sourced BOM and calculation notes
Parts:
- added C44: 100n, symbol Device:C_Small
- added U2: TPS3808G33DBVR, Package_TO_SOT_SMD:SOT-23-6, symbol Power_Devices:TPS3808G33DBVR
Connections:
- net +3V3_MCU: now also C44.1, U2.5 (SENSE), U2.6 (VDD)
- net GND: now also C44.2, U2.2 (GND)
- net MCU_RESET_N: now also U2.1 (~{RESET}); no longer SW1.1
- new net SW_RESET_N: SW1.1, U2.3 (~{MR})
- no-connect marks 1 -> 2
Other:
- note added: "RST-001: U2 supervises +3V3_MCU; SW1 asserts MR. CT open: release delay 12..28 ms; 12/2.4 = 5x MCU minimum. Falling threshold = 3.07*(1 +/- 0.015) = 3.02395..3.11605 V. Conservative release screen = 3.11605*1.025 = 3.19395125 V. ASSUMED rail +/-2%: 3.3*0.98 - 3.19395125 = 40.05 mV margin. R1 worst pull-up current = 3.6/9900 = 0.364 mA < 1 mA. RES low margin = 0.2*3.02395 - 0.4 = 0.20479 V. No RES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"
- note removed: "NO capacitor on RES: it must track VCC for internal POR. External reset drivers must be open-drain/open-collector. Hold RESET low >= 3 ms, then release after VCC is valid. Hold BOOT during external reset release for SCI/USBFS mode. Normal MD high; SWD/JTAG boot requests occur during RES low. Device lifecycle / authentication restrictions still apply."

Commit message: Connect radio reset controls through schematic hierarchy
Changed lines of the file:
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@@
+	(wire
+		(pts
+			(xy 129.54 203.2) (xy 129.54 210.82)
+		)
+		(stroke
+			(width 0)
+			(type default)
+		)
+	)
 	(wire
 		(pts
@@
 		(effects
 			(font
+				(size 1.27 1.27)
+			)
+			(justify left)
+		)
+	)
+	(hierarchical_label "MCU_RESET_N"
+		(shape output)
+		(at 129.54 210.82 0)
+		(effects
+			(font

Commit message: Replace engineering BOOT and reset switches with internal service pads
Parts:
- TP1: renamed from SW1; value RESET -> RESET_SERVICE; symbol Switch:SW_Push -> Connector:TestPoint_2Pole; Procurement_Status TBD - source normally-open momentary switch; mechanical cho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 -> (none); now left out of the parts list
- TP2: renamed from SW2; value BOOT -> BOOT_SERVICE; symbol Switch:SW_Push -> Connector:TestPoint_2Pole; Procurement_Status TBD - source normally-open momentary switch; mechanical cho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 -> (none); now left out of the parts list
Other:
- note added: "RST-001: U2 supervises +3V3_MCU; TP1 is internal MR service access. CT open: release delay 12..28 ms; 12/2.4 = 5x MCU minimum. Falling threshold = 3.07*(1 +/- 0.015) = 3.02395..3.11605 V. Conservative release screen = 3.11605*1.025 = 3.19395125 V. ASSUMED rail +/-2%: 3.3*0.98 - 3.19395125 = 40.05 mV margin. R1 worst pull-up current = 3.6/9900 = 0.364 mA < 1 mA. RES low margin = 0.2*3.02395 - 0.4 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"
- note removed: "RST-001: U2 supervises +3V3_MCU; SW1 asserts MR. CT open: release delay 12..28 ms; 12/2.4 = 5x MCU minimum. Falling threshold = 3.07*(1 +/- 0.015) = 3.02395..3.11605 V. Conservative release screen = 3.11605*1.025 = 3.19395125 V. ASSUMED rail +/-2%: 3.3*0.98 - 3.19395125 = 40.05 mV margin. R1 worst pull-up current = 3.6/9900 = 0.364 mA < 1 mA. RES low margin = 0.2*3.02395 - 0.4 = 0.20479 V. No RES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"
Changed lines of the file:
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@@
 		)
 	)
-	(text "RST-001: U2 supervises +3V3_MCU; SW1 asserts MR.\nCT open: release delay 12..28 ms; 12/2.4 = 5x MCU minimum.\nFalling threshold = 3.07*(1 +/- 0.015) = 3.02395..3.11605 V.\nConservative release screen = 3.11605*1.025 = 3.19395125 V.\nASSUMED rail +/-2%: 3.3*0.98 - 3.19395125 = 40.05 mV margin.\nR1 worst pull-up current = 3.6/9900 = 0.364 mA < 1 mA.\nRES low margin = 0.2*3.02395 - 0.4 = 0.20479 V.\nNo RES capacitor; open-drain reset drivers only.\nExternal RES startup path; do not assume internal POR flag.\nFull math, limits and Python: design/boot_and_debug.md RST-001."
+	(text "RST-001: U2 supervises +3V3_MCU; TP1 is internal MR service access.\nCT open: release delay 12..28 ms; 12/2.4 = 5x MCU minimum.\nFalling threshold = 3.07*(1 +/- 0.015) = 3.02395..3.11605 V.\nConservative release screen = 3.11605*1.025 = 3.19395125 V.\nASSUMED rail +/-2%: 3.3*0.98 - 3.19395125 = 40.05 mV margin.\nR1 worst pull-up current = 3.6/9900 = 0.364 mA < 1 mA.\nRES low margin = 0.2*3.02395 - 0.4 = 0.20479 V.\nNo RES capacitor; open-drain reset drivers only.\nExternal RES startup path; do not assume internal POR flag.\nFull math, limits and Python: design/boot_and_debug.md RST-001.	"
 		(exclude_from_sim no)
 		(at 25.4 223.52 0)
@@
 	)
 	(symbol
-		(lib_id "Switch:SW_Push")
+		(lib_id "Connector:TestPoint_2Pole")
 		(at 139.7 162.56 0)
 		(unit 1)
 		(body_style 1)
 		(exclude_from_sim no)
-		(in_bom yes)
+		(in_bom no)
 		(on_board yes)
-		(in_pos_files yes)
+		(in_pos_files no)
 		(dnp no)
-		(property "Reference" "SW2"
-			(at 140.97 160.02 0)
+		(property "Reference" "TP2"
+			(at 139.7 161.036 0)
 			(show_name no)
 			(do_not_autoplace no)
@@
 					(size 1.27 1.27)
 				)
-				(justify left)
 			)
 		)
-		(property "Value" "BOOT"
-			(at 139.7 164.084 0)
+		(property "Value" "BOOT_SERVICE"
+			(at 139.7 164.338 0)
 			(show_name no)
 			(do_not_autoplace no)
@@
 		)
 		(property "Footprint" ""
-			(at 139.7 157.48 0)
-			(hide yes)
-			(show_name no)
-			(do_not_autoplace no)
-			(effects
-				(font
-					(size 1.27 1.27)
-				)
-			)
-		)
-		(property "Datasheet" ""
-			(at 139.7 157.48 0)
-			(hide yes)
-			(show_name no)
-			(do_not_autoplace no)
-			(effects
-				(font
-					(size 1.27 1.27)
-				)
-			)
-		)
-		(property "Description" "Push button switch, generic, two pins"
 			(at 139.7 162.56 0)
 			(hide yes)
@@
 			)
 		)
-		(property "ki_keywords" "switch normally-open pushbutton push-button"
-			(at 139.7 162.56 0)
-			(hide yes)
-			(show_name no)
-			(do_not_autoplace no)
-			(effects
-				(font
-					(size 1.27 1.27)
-				)
-			)
-		)
-		(property "DigiKey_Part_Number" ""
-			(at 139.7 162.56 0)
-			(hide yes)
-			(show_name no)
-			(do_not_autoplace no)
-			(effects
-				(font
-					(size 1.27 1.27)
-				)
-			)
-		)
-		(property "DigiKey_URL" ""
-			(at 139.7 162.56 0)
-			(hide yes)
-			(show_name no)
-			(do_not_autoplace no)
-			(effects
-				(font
-					(size 1.27 1.27)
-				)
-			)
-		)
-		(property "Procurement_Status" "TBD - source normally-open momentary switch; mechanical choice pending"
-			(at 139.7 162.56 0)
-			(hide yes)
-			(show_name no)
-			(do_not_autoplace no)
-			(effects
-				(font
-					(size 1.27 1.27)
-				)
-			)
-		)
-		(property "Sourcing_Snapshot" ""
+		(property "Datasheet" ""
 			(at 139.7 162.56 0)
 			(hide yes)
@@
 			)
 		)
-		(property "Mouser_URL" ""
+		(property "Description" "Internal paired copper service pads: 1=MCU_BOOT_MD, 2=GND. Fixture holds MD low while asserting and releasing external RES for SCI/USB ROM boot. No fitted switch. HUM 4.3-4.4."
 			(at 139.7 162.56 0)
 			(hide yes)
@@
 			(project "ereader_rev1"
 				(path "/0586cc51-9c57-495b-a0c9-c29ba0d48166/29d11a66-d141-4e93-8408-b9f3c692a4bc"
-					(reference "SW2")
+					(reference "TP2")
 					(unit 1)
 				)
@@
 	)
 	(symbol
-		(lib_id "Switch:SW_Push")
+		(lib_id "Connector:TestPoint_2Pole")
 		(at 66.04 162.56 0)
 		(unit 1)
 		(body_style 1)
 		(exclude_from_sim no)
-		(in_bom yes)
+		(in_bom no)
 		(on_board yes)
-		(in_pos_files yes)
+		(in_pos_files no)
 		(dnp no)
-		(property "Reference" "SW1"
-			(at 67.31 160.02 0)
+		(property "Reference" "TP1"
+			(at 66.04 161.036 0)
 			(show_name no)
 			(do_not_autoplace no)
@@
 					(size 1.27 1.27)
 				)
-				(justify left)
 			)
 		)
-		(property "Value" "RESET"
-			(at 66.04 164.084 0)
+		(property "Value" "RESET_SERVICE"
+			(at 66.04 164.338 0)
 			(show_name no)
 			(do_not_autoplace no)
@@
 		)
 		(property "Footprint" ""
-			(at 66.04 157.48 0)
-			(hide yes)
-			(show_name no)
-			(do_not_autoplace no)
-			(effects
-				(font
-					(size 1.27 1.27)
-				)
-			)
-		)
-		(property "Datasheet" ""
-			(at 66.04 157.48 0)
-			(hide yes)
-			(show_name no)
-			(do_not_autoplace no)
-			(effects
-				(font
-					(size 1.27 1.27)
-				)
-			)
-		)
-		(property "Description" "Push button switch, generic, two pins"
 			(at 66.04 162.56 0)
 			(hide yes)
@@
 			)
 		)
-		(property "ki_keywords" "switch normally-open pushbutton push-button"
-			(at 66.04 162.56 0)
-			(hide yes)
-			(show_name no)
-			(do_not_autoplace no)
-			(effects
-				(font
-					(size 1.27 1.27)
-				)
-			)
-		)
-		(property "DigiKey_Part_Number" ""
-			(at 66.04 162.56 0)
-			(hide yes)
-			(show_name no)
-			(do_not_autoplace no)
-			(effects
-				(font
-					(size 1.27 1.27)
-				)
-			)
-		)
-		(property "DigiKey_URL" ""
-			(at 66.04 162.56 0)
-			(hide yes)
-			(show_name no)
-			(do_not_autoplace no)
-			(effects
-				(font
-					(size 1.27 1.27)
-				)
-			)
-		)
-		(property "Procurement_Status" "TBD - source normally-open momentary switch; mechanical choice pending"
-			(at 66.04 162.56 0)
-			(hide yes)
-			(show_name no)
-			(do_not_autoplace no)
-			(effects
-				(font
-					(size 1.27 1.27)
-				)
-			)
-		)
-		(property "Sourcing_Snapshot" ""
+		(property "Datasheet" ""
 			(at 66.04 162.56 0)
 			(hide yes)
@@
 			)
 		)
-		(property "Mouser_URL" ""
+		(property "Description" "Internal paired copper service pads: 1=supervisor MR, 2=GND. Shorting pads asserts MCU reset through U2; direct debugger reset remains J1.10. No fitted switch. RST-001."
 			(at 66.04 162.56 0)
 			(hide yes)
@@
 			(project "ereader_rev1"
 				(path "/0586cc51-9c57-495b-a0c9-c29ba0d48166/29d11a66-d141-4e93-8408-b9f3c692a4bc"
-					(reference "SW1")
+					(reference "TP1")
 					(unit 1)
 				)

Commit message: Complete MCU reset checkpoint and portable engineering records
Refs #825, #826, #846. Preserve the unresolved radio release margin and unfinished schematic status; refresh full PDF and native BOM.
Parts:
- added C95: 10n, symbol Device:C_Small
- added R67: 33k, symbol Device:R
- added R74: 20k, symbol Device:R
- added R75: 10k, symbol Device:R
- U2: value TPS3808G33DBVR -> TPS389001DSET; footprint Package_TO_SOT_SMD:SOT-23-6 -> (none); symbol Power_Devices:TPS3808G33DBVR -> Power_Devices:TPS389001DSET; DigiKey_Part_Number 296-17195-1-ND -> 296-44489-1-ND; DigiKey_URL https://www.digikey.com/en/products/detail/texas-instruments/TPS3808G33DBVR/666727 -> https://www.digikey.com/en/products/detail/texas-instruments/TPS389001DSET/6110554; Manufacturer_Part_Number TPS3808G33DBVR -> TPS389001DSET; Procurement_Status Selected - TI active production; RST-001 electrical screeni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 -> Selected and wired for conditional DC/startup coordination;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; Selection_Basis RST-001: 3.07 V fixed threshold, CT-open 12..28 ms delay, o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 -> RST-002: adjustable 1.15V falling/1.157V rising supervisor,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; Sourcing_Snapshot 2026-09-05: DigiKey 22054 stock; USD 1.84/1.355/1.0984 at q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 -> 2026-09-08 DigiKey: 2090 stock; USD 2.22/1.643/1.3395 at 1/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
Connections:
- net +3V3_MCU: now also U2.4 (VDD), R67.1, R75.1; no longer U2.5 (SENSE), U2.6 (VDD)
- net GND: now also C95.2, R74.2
- net MCU_RESET_N: now also U2.6 (~{RESET}); no longer U2.1 (~{RESET})
- net SW_RESET_N: now also R75.2
- new net: C95.1, U2.5 (CT)
- new net: R67.2, R74.1, U2.1 (SENSE)
- no-connect marks 2 -> 1
Other:
- note added: "RST-002: U2 TPS389001DSET; R67=33k, R74=20k, R75=10k, C95=10n. Sense resistors: +/-0.05%, 10ppm/C over 100C, allocated +/-0.15% assembly/aging. fL=.9995*.999*.9985=.99700274925; fH=1.0005*1.001*1.0015=1.00300275075. Klo=1+33000*fL/(20000*fH); Khi=1+33000*fH/(20000*fL); E=150nA*33000*fH. Vfall=1.15*.99*Klo-E .. 1.15*1.01*Khi+E = 3.000822727..3.094473285V. Vrise=1.157*.99*Klo-E .. 1.157*1.01*Khi+E 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"
- note removed: "RST-001: U2 supervises +3V3_MCU; TP1 is internal MR service access. CT open: release delay 12..28 ms; 12/2.4 = 5x MCU minimum. Falling threshold = 3.07*(1 +/- 0.015) = 3.02395..3.11605 V. Conservative release screen = 3.11605*1.025 = 3.19395125 V. ASSUMED rail +/-2%: 3.3*0.98 - 3.19395125 = 40.05 mV margin. R1 worst pull-up current = 3.6/9900 = 0.364 mA < 1 mA. RES low margin = 0.2*3.02395 - 0.4 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"
- moved on the sheet: U2
