File: ra8p1_kicad/ereader/power_button.kicad_sch (KiCad schematic)
At the start: 11 parts, among them SW1 POWER, U9 LTC2954ITS8-1

Commit message: Add reviewed e-reader held-control supply
Place reverse isolation, output charging resistor and four-capacitor reservoir. Sense the held side to detect current-limited source collapse, and budget pre-trip reverse current explicitly.

Include native BOM, linked Python-checked calculations and refreshed eight-page schematic PDF. Exact netlist and visual checks pass; independent review corrected one topology fault. ERC remains at the existing 204 errors and two warnings while source, supervision and discharge circuits are unfinished.
Parts:
- added C62: 100n, symbol Device:C_Small
- added C63, C64, C65, C66: 100u, symbol Device:C_Polarized_Small
- added R31: 100R, symbol Device:R
- added U10: LM66100DCKR, Package_TO_SOT_SMD:SOT-363_SC-70-6, symbol Power_Management:LM66100DCK
Connections:
- net GND: now also C62.2, C63.2, C64.2, C65.2, C66.2, U10.2 (GND), U10.5 (ST)
- net SYS_AON: now also C62.1, U10.1 (VIN); no longer C55.1, U9.1 (VIN)
- new net: R31.1, U10.6 (VOUT)
- new net AON_HOLD: C55.1, C63.1, C64.1, C65.1, C66.1, R31.2, U10.3 (~{CE}), U9.1 (VIN)
Other:
- note added: "ERC supply path: U10 VOUT through R31. PWR_FLAG declares that series-fed source only; raw SYS_AON source remains unimplemented."
- note added: "INCOMPLETE POWER CONTROL - NOT FOR FABRICATION PB, INT, KILL and held-supply reservoir are connected. SYS_AON has no source; U9 EN has no load or pull-up yet. Source supervision and rail discharge remain to be implemented. Power-control operation is not yet complete or qualified. Implementation and qualification: ../design/system_power_design.md SYS-007; button calculations: ../design/single_butt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"
- note added: "SYS-007 REVISED: HELD SUPPLY / U10, R31, C62-C66 C63-C66: 4 x 100uF/10V; Cmin=400uF*0.9^3=291.6uF. VIN=raw SYS; VOUT->R31->reservoir; CE senses reservoir. Icontrol<=1.125mA incl 500uA bank leakage allocation. Pre-trip reverse: 80mV/98.01ohm<0.817mA. Itotal=1.942mA. Vinitial=3.263705831-max(0.250,0.001125*102.24) =3.013705831V (threshold OR resistive-drop limit). t_hold=[291.6uF*(3.013705831-2.7)V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"
- note removed: "INCOMPLETE POWER CONTROL - NOT FOR FABRICATION PB input, INT and KILL interfaces are placed and connected. SYS_AON has no source; U9 EN has no load or pull-up yet. Held supply, source supervision and rail discharge are pending. This sheet does not yet implement functional product power control. Implementation and qualification: ../design/system_power_design.md SYS-007; button calculations: ../des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"

Commit message: Add reviewed e-reader source supervisor and enable network
Parts:
- added C67, C69, C70, C71: 100n, symbol Device:C_Small
- added C68: 1n, symbol Device:C_Small
- added R32: 732k, symbol Device:R
- added R33, R34: 100k, symbol Device:R
- added U11: TPS3808G01DBVR, Package_TO_SOT_SMD:SOT-23-6, symbol Power_Devices:TPS3808G01DBVR
Connections:
- net AON_HOLD: now also C67.1, R34.1, U11.3 (~{MR}), U11.6 (VDD)
- net GND: now also C67.2, C68.2, C69.2, C70.2, C71.2, R33.2, U11.2 (GND)
- net SYS_AON: now also R32.1
- net MAIN_PWR_EN: now reaches U9.6 (EN)
- net MAIN_PWR_EN: now also R34.2, U11.1 (~{RESET})
- new net: C68.1, R32.2, R33.1, U11.5 (SENSE)
- new net: C69.1, C70.1, C71.1, U11.4 (CT)
Other:
- note added: "INCOMPLETE POWER CONTROL - NOT FOR FABRICATION PB, INT, KILL, held supply and source supervisor are connected. SYS_AON has no source; MAIN_PWR_EN has no converter load yet. Fault-to-KILL clamp and main-rail discharge remain to be implemented. Power-control operation is not yet complete or qualified. Implementation and qualification: ../design/system_power_design.md SYS-007; button calculations: .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"
- note added: "SYS-007: SOURCE SUPERVISION / U11, R32-R34, C67-C71 Vtrip=Vref*(1+R32/R33)+Isense*R32. Nominal=0.405*(1+732k/100k)=3.369600V. Vref +/-2%, Isense +/-25nA; each R +/-0.1%, 25ppm/C, 100C. Corner trip=3.263705831..3.476597632V. C68: tau=(732k||100k)*1n=87.980769us (nominal). C69-C71: 3x100n C0G; initial/temp=284.145..316.827nF. CT delay=300/175+0.0005=1.714786s nominal. 0.6*(284.145/175+0.0005)=0.974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"
- note removed: "INCOMPLETE POWER CONTROL - NOT FOR FABRICATION PB, INT, KILL and held-supply reservoir are connected. SYS_AON has no source; U9 EN has no load or pull-up yet. Source supervision and rail discharge remain to be implemented. Power-control operation is not yet complete or qualified. Implementation and qualification: ../design/system_power_design.md SYS-007; button calculations: ../design/single_butt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"

Commit message: Add reviewed e-reader shutdown clamp and rail discharge
Parts:
- added C72: 100n, symbol Device:C_Small
- added Q1, Q2: DMN2056U-7, Package_TO_SOT_SMD:SOT-23, symbol Transistor_FET:DMN2056U
- added R35, R36: 1k, symbol Device:R
- added R37, R38: 1M, symbol Device:R
- added R39, R40: 22R, symbol Device:R
- added U12: 74LVC1G14GW,125, symbol 74xGxx:74LVC1G14
Connections:
- net +3V3_MCU: now also R39.2, R40.2
- net AON_HOLD: now also C72.1, U12.5 (VCC)
- net GND: now also C72.2, Q1.2 (S), Q2.2 (S), R37.1, R38.1, U12.3 (GND)
- net MAIN_PWR_EN: now also U12.2
- net POWER_KILL_N: now also Q1.3 (D)
- new net: Q1.1 (G), R35.2, R37.2
- new net: Q2.1 (G), R36.2, R38.2
- new net: Q2.3 (D), R39.1, R40.1
- new net POWER_OFF_H: R35.1, R36.1, U12.4
Other:
- note added: "INCOMPLETE POWER CONTROL - NOT FOR FABRICATION PB, INT, KILL, held supply and source supervisor are connected. U12/Q1/Q2 now provide fault KILL clamp and main-rail discharge. SYS_AON has no source; MAIN_PWR_EN has no converter load yet. USB permission-latch clear and source/converter blocks remain. Power-control operation is not yet complete or qualified. Engineering basis and tests: ../design/sy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"
- note added: "SYS-007: SHUTDOWN / U12, Q1-Q2, R35-R40, C72 POWER_OFF_H=NOT(MAIN_PWR_EN); held-domain VCC=2.7..4.6V. R35/R36=1k; R37/R38=1M; 1% + 100ppm/C over 100C. 3-gate peak<=3*4.6/(1000*0.99^2)=14.080196mA <50mA. Includes future USB-clear gate; static<=17.080196uA <100uA. VGSmin=(2.6-1020.1*1uA)/(1+1020.1/980100)=2.596278V. 1uA per gate/board leakage is a qualification allocation. R39||R40 + Q2: Rmax=22*1.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"
- note removed: "INCOMPLETE POWER CONTROL - NOT FOR FABRICATION PB, INT, KILL, held supply and source supervisor are connected. SYS_AON has no source; MAIN_PWR_EN has no converter load yet. Fault-to-KILL clamp and main-rail discharge remain to be implemented. Power-control operation is not yet complete or qualified. Implementation and qualification: ../design/system_power_design.md SYS-007; button calculations: .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"

Commit message: Implement main digital supply with linked engineering calculations
Wire the TPS63802 converter and its hierarchical enable, source its exact BOM, and refresh the full nine-page schematic PDF. Preserve the SDRAM pin and timing contract for the memory implementation. Track #825 and #827; system qualification remains open.
Other:
- note added: "INCOMPLETE POWER CONTROL - NOT FOR FABRICATION PB, INT, KILL, held supply and source supervisor are connected. U12/Q1/Q2 provide fault KILL clamp and main-rail discharge. MAIN_PWR_EN now controls U13 on Main 3V3 digital supply. SYS_AON source and USB permission-latch clear remain to be built. Power-control operation is not yet complete or qualified. Engineering: ../design/system_power_design.md S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"
- note removed: "INCOMPLETE POWER CONTROL - NOT FOR FABRICATION PB, INT, KILL, held supply and source supervisor are connected. U12/Q1/Q2 now provide fault KILL clamp and main-rail discharge. SYS_AON has no source; MAIN_PWR_EN has no converter load yet. USB permission-latch clear and source/converter blocks remain. Power-control operation is not yet complete or qualified. Engineering basis and tests: ../design/sy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"
Changed lines of the file:
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@@
 		)
 	)
-	(text "INCOMPLETE POWER CONTROL - NOT FOR FABRICATION\nPB, INT, KILL, held supply and source supervisor are connected.\nU12/Q1/Q2 now provide fault KILL clamp and main-rail discharge.\nSYS_AON has no source; MAIN_PWR_EN has no converter load yet.\nUSB permission-latch clear and source/converter blocks remain.\nPower-control operation is not yet complete or qualified.\nEngineering basis and tests: ../design/system_power_design.md SYS-007."
+	(text "INCOMPLETE POWER CONTROL - NOT FOR FABRICATION\nPB, INT, KILL, held supply and source supervisor are connected.\nU12/Q1/Q2 provide fault KILL clamp and main-rail discharge.\nMAIN_PWR_EN now controls U13 on Main 3V3 digital supply.\nSYS_AON source and USB permission-latch clear remain to be built.\nPower-control operation is not yet complete or qualified.\nEngineering: ../design/system_power_design.md SYS-007;\nconverter math: ../design/power_decoupling.md PWR-002/PWR-003."
 		(exclude_from_sim no)
 		(at 228.6 50.8 0)
@@
 		)
 	)
-	(label "MAIN_PWR_EN"
-		(at 129.54 60.96 0)
-		(effects
-			(font
-				(size 1.27 1.27)
-			)
-			(justify left bottom)
-		)
-	)
 	(label "POWER_OFF_H"
 		(at 231.14 233.68 0)
@@
 		)
 	)
+	(hierarchical_label "MAIN_PWR_EN"
+		(shape output)
+		(at 129.54 60.96 0)
+		(effects
+			(font
+				(size 1.27 1.27)
+			)
+			(justify left)
+		)
+	)
 	(symbol
 		(lib_id "power:GND")
@@
 		(in_pos_files yes)
 		(dnp no)
-		(fields_autoplaced yes)
 		(property "Reference" "U9"
-			(at 116.4433 59.69 0)
+			(at 116.84 54.61 0)
 			(show_name no)
 			(do_not_autoplace no)
@@
 		)
 		(property "Value" "LTC2954ITS8-1"
-			(at 116.4433 62.23 0)
+			(at 116.84 57.15 0)
 			(show_name no)
 			(do_not_autoplace no)

Commit message: Wire LTC3119 power-stage draft and held RUN control
Add native RUN buffer and held-domain clamp with verified connectivity, sourced BOM fields, and linked PWR-004 calculations. Export the full schematic PDF and native BOM.

Keep rail adoption blocked by SDRAM logic-high conflict #846. Whole-project ERC remains 133 errors and two warnings; this checkpoint adds no findings.
Parts:
- R34: value 100k -> 110k; DigiKey_Part_Number 311-100KHRCT-ND -> 311-110KHRCT-ND; DigiKey_URL https://www.digikey.com/en/products/detail/yageo/RC0603FR-07100KL/729836 -> https://www.digikey.com/en/products/detail/yageo/RC0603FR-07110KL/726905; Manufacturer_Part_Number RC0603FR-07100KL -> RC0603FR-07110KL; Procurement_Status Selected - electrical ratings and sourcing checked; footpri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 -> Active; DigiKey stock checked 2026-09-08; unreserved; reche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; Selection_Basis SYS-007: 100k EN pullup AON_HOLD to MAIN_PWR_EN. Allocate 3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 -> PWR-004: 110k AON_HOLD-to-MAIN_PWR_EN pull-up; 1% initial p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; Sourcing_Snapshot 2026-09-07: DigiKey stock 2200236; USD 0.10/0.025/0.0122 at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 -> 2026-09-08: DigiKey 214574 in stock; USD 0.10 at 1; unreser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
- R35, R36: Selection_Basis SYS-007: 1k per held-domain gate; Rmin=980.1R, Rmax=1020.1R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 -> SYS-007 / PWR-004: 1k per held-domain gate; R=980.1..1020.1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
- R39, R40: Selection_Basis SYS-007: two 22R 1W in parallel, Rpath_max=11.4211R with 0.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 -> SYS-007 / PWR-004: two 22R 1W in parallel, Rpath_max=11.421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
- U12: Selection_Basis SYS-007: 2.7-4.6V held-domain inverter; 1uA input leakage; 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 -> SYS-007 / PWR-004: 2.7..4.6V held-domain inverter; 1uA inpu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
Other:
- note added: "INCOMPLETE POWER CONTROL - NOT FOR FABRICATION PB, INT, KILL, held supply and source supervisor are connected. U12/Q1/Q2 provide fault KILL clamp and main-rail discharge. MAIN_PWR_EN feeds raw U16; held Q3 separately clamps U13 RUN. SYS_AON source and USB permission-latch clear remain to be built. Power-control operation is not yet complete or qualified. Current converter/control draft: ../design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"
- note added: "SYS-007 / PWR-004: HELD SUPPLY / U10, R31, C62-C66 C63-C66: 4 x 100uF/10V; Cmin=400uF*0.9^3=291.6uF. VIN=raw SYS; VOUT->R31->reservoir; CE senses reservoir. Icontrol<=1.125mA incl 500uA bank leakage allocation. Pre-trip reverse: 80mV/98.01ohm<0.817mA. Itotal=1.942mA. Vinitial=3.263705831-max(0.250,0.001125*102.24) =3.013705831V (threshold OR resistive-drop limit). t_hold=[291.6uF*(3.013705831-2.7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"
- note added: "SYS-007 / PWR-004: SHUTDOWN / U12, Q1-Q3, R35-R40, R70-R71 POWER_OFF_H=NOT(MAIN_PWR_EN); held-domain VCC=2.7..4.6V. Each gate branch: 1k series / 1M pulldown; 1% + 100ppm/C, 100C. 4-gate peak<=4*4.6/(1000*0.99^2)=18.773595mA <50mA. Includes future USB-clear; static<=22.773595uA <100uA. VGSmin=(2.6-1020.1*1uA)/(1+1020.1/980100)=2.596278V. 1uA per gate/board leakage is a qualification allocation. R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"
- note added: "SYS-007 / PWR-004: SOURCE SUPERVISION / U11, R32-R34, C67-C71 Vtrip=Vref*(1+R32/R33)+Isense*R32. Nominal=0.405*(1+732k/100k)=3.369600V. Vref +/-2%, Isense +/-25nA; each R +/-0.1%, 25ppm/C, 100C. Corner trip=3.263705831..3.476597632V. C68: tau=(732k||100k)*1n=87.980769us (nominal). C69-C71: 3x100n C0G; initial/temp=284.145..316.827nF. CT delay=300/175+0.0005=1.714786s nominal. 0.6*(284.145/175+0.0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"
- note removed: "INCOMPLETE POWER CONTROL - NOT FOR FABRICATION PB, INT, KILL, held supply and source supervisor are connected. U12/Q1/Q2 provide fault KILL clamp and main-rail discharge. MAIN_PWR_EN now controls U13 on Main 3V3 digital supply. SYS_AON source and USB permission-latch clear remain to be built. Power-control operation is not yet complete or qualified. Engineering: ../design/system_power_design.md S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"
- note removed: "SYS-007 REVISED: HELD SUPPLY / U10, R31, C62-C66 C63-C66: 4 x 100uF/10V; Cmin=400uF*0.9^3=291.6uF. VIN=raw SYS; VOUT->R31->reservoir; CE senses reservoir. Icontrol<=1.125mA incl 500uA bank leakage allocation. Pre-trip reverse: 80mV/98.01ohm<0.817mA. Itotal=1.942mA. Vinitial=3.263705831-max(0.250,0.001125*102.24) =3.013705831V (threshold OR resistive-drop limit). t_hold=[291.6uF*(3.013705831-2.7)V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"
- note removed: "SYS-007: SHUTDOWN / U12, Q1-Q2, R35-R40, C72 POWER_OFF_H=NOT(MAIN_PWR_EN); held-domain VCC=2.7..4.6V. R35/R36=1k; R37/R38=1M; 1% + 100ppm/C over 100C. 3-gate peak<=3*4.6/(1000*0.99^2)=14.080196mA <50mA. Includes future USB-clear gate; static<=17.080196uA <100uA. VGSmin=(2.6-1020.1*1uA)/(1+1020.1/980100)=2.596278V. 1uA per gate/board leakage is a qualification allocation. R39||R40 + Q2: Rmax=22*1.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"
- note removed: "SYS-007: SOURCE SUPERVISION / U11, R32-R34, C67-C71 Vtrip=Vref*(1+R32/R33)+Isense*R32. Nominal=0.405*(1+732k/100k)=3.369600V. Vref +/-2%, Isense +/-25nA; each R +/-0.1%, 25ppm/C, 100C. Corner trip=3.263705831..3.476597632V. C68: tau=(732k||100k)*1n=87.980769us (nominal). C69-C71: 3x100n C0G; initial/temp=284.145..316.827nF. CT delay=300/175+0.0005=1.714786s nominal. 0.6*(284.145/175+0.0005)=0.974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"
